File: ufc_panel.kicad_pcb (KiCad board)
At the start: 2 copper layers, 252 x 58 mm, 101 parts, among them J1 Conn_01x20_Socket, Q1 BC817-25LT1G, SW1 SW_Push_45deg, SW10 SW_Push_45deg, SW11 SW_Push_45deg, SW12 SW_Push_45deg, SW13 SW_Push_45deg, SW14 SW_Push_45deg, SW15 SW_Push_45deg, SW16 SW_Push_45deg, SW17 SW_Push_45deg, SW18 SW_Push_45deg, SW19 SW_Push_45deg, SW2 SW_Push_45deg, SW20 SW_Push_45deg, SW21 SW_Push_45deg, SW22 SW_Push_45deg, SW23 SW_Push_45deg, SW24 SW_Push_45deg, SW25 SW_Push_45deg, SW26 SW_Push_45deg, SW27 SW_Push_45deg, SW28 SW_Push_45deg, SW29 SW_Push_45deg, SW3 SW_Push_45deg, SW30 SW_Push_45deg, SW31 SW_Push_45deg, SW32 SW_Push_45deg, SW33 SW_Push_45deg, SW34 SW_Push_45deg, SW35 SW_Push_45deg, SW4 SW_Push_45deg, SW5 SW_Push_45deg, SW6 SW_Push_45deg, SW7 SW_Push_45deg, SW8 SW_Push_45deg, SW9 SW_Push_45deg

Commit message: feat: new version - v1.1; redesigned traces, connector, etc
Parts:
- removed the D26 at (190.2, 72.2)
- removed the LED8 at (131.9, 55.8)
- removed the R6 at (98.9, 56.0)
- removed the SW27 at (177.9, 27.8)
- removed the SW30 at (236.8, 26.9)
- removed the SW32 at (225.7, 60.5)
- added D32: D_Small, Diode_SMD:D_SOD-123, B.Cu at (195.0, 60.4)
- added LED15: HSMY-C150, LED_SMD:LED_1206_3216Metric_Pad1.42x1.75mm_HandSolder, F.Cu at (176.5, 25.8)
- added R16: 3300, Resistor_SMD:R_0603_1608Metric, F.Cu at (261.8, 28.6)
- added SW34: Switch, Custom_Footprint_Switches:SW_PUSH_6mm_H4.3mm_INT_CONNECTED, F.Cu at (237.9, 67.6)
- added SW7: Switch, Custom_Footprint_Switches:SW_PUSH_6mm_H4.3mm_INT_CONNECTED, F.Cu at (180.7, 29.1)
- added SW9: Switch, Custom_Footprint_Switches:SW_PUSH_6mm_H4.3mm_INT_CONNECTED, F.Cu at (240.6, 28.3)
- D1: renamed from D5; moved to B.Cu
- D10: renamed from D15; moved to B.Cu
- D11: renamed from D16; moved to B.Cu
- D12: renamed from D11; moved to B.Cu
- D13: renamed from D18; moved to B.Cu
- D14: renamed from D17; moved to B.Cu
- D15: renamed from D12; moved to B.Cu
- D16: renamed from D19; moved to B.Cu
- D17: renamed from D13; moved to B.Cu
- D18: renamed from D14; moved to B.Cu
- D19: renamed from D8; moved to B.Cu
- D2, D24, D29, D31, D34: moved to B.Cu
- D20: renamed from D28; moved to B.Cu
- D21: renamed from D30; moved to B.Cu
- D22: renamed from D27; moved to B.Cu
- D23: renamed from D20; moved to B.Cu
- D25: renamed from D21; moved to B.Cu
- D26: renamed from D25; moved to B.Cu
- D27: renamed from D23; moved to B.Cu
- D28: renamed from D22; moved to B.Cu
- D3: renamed from D10; moved to B.Cu
- D30: renamed from D32; moved to B.Cu
- D33: renamed from D35; moved to B.Cu
- D35: renamed from D33; moved to B.Cu
- D4: renamed from D3; moved to B.Cu
- D5: renamed from D4; moved to B.Cu
- D6: renamed from D1; moved to B.Cu
- D7: renamed from D9; moved to B.Cu
- D8: renamed from D6; moved to B.Cu
- D9: renamed from D7; moved to B.Cu
- J1: value Conn_01x20_Socket -> Conn_2x10 Socket; footprint Connector_PinHeader_1.00mm:PinHeader_2x10_P1.00mm_Vertical -> Connector_PinHeader_2.54mm:PinHeader_1x20_P2.54mm_Vertical
- LED1: renamed from LED2; footprint MOUSER:LEDC3216X120N -> LED_SMD:LED_1206_3216Metric_Pad1.42x1.75mm_HandSolder
- LED10: renamed from LED13; footprint MOUSER:LEDC3216X120N -> LED_SMD:LED_1206_3216Metric_Pad1.42x1.75mm_HandSolder
- LED11: renamed from LED12; footprint MOUSER:LEDC3216X120N -> LED_SMD:LED_1206_3216Metric_Pad1.42x1.75mm_HandSolder
- LED12: renamed from LED10; footprint MOUSER:LEDC3216X120N -> LED_SMD:LED_1206_3216Metric_Pad1.42x1.75mm_HandSolder
- LED13: renamed from LED6; footprint MOUSER:LEDC3216X120N -> LED_SMD:LED_1206_3216Metric_Pad1.42x1.75mm_HandSolder
- LED2: renamed from LED1; footprint MOUSER:LEDC3216X120N -> LED_SMD:LED_1206_3216Metric_Pad1.42x1.75mm_HandSolder
- LED3: renamed from LED4; footprint MOUSER:LEDC3216X120N -> LED_SMD:LED_1206_3216Metric_Pad1.42x1.75mm_HandSolder
- LED4: renamed from LED3; footprint MOUSER:LEDC3216X120N -> LED_SMD:LED_1206_3216Metric_Pad1.42x1.75mm_HandSolder
- LED5: renamed from LED9; footprint MOUSER:LEDC3216X120N -> LED_SMD:LED_1206_3216Metric_Pad1.42x1.75mm_HandSolder
- LED6: renamed from LED5; footprint MOUSER:LEDC3216X120N -> LED_SMD:LED_1206_3216Metric_Pad1.42x1.75mm_HandSolder
- LED7: renamed from LED14; value HSMY-C150 -> HSMG-C150; footprint MOUSER:LEDC3216X120N -> LED_SMD:LED_1206_3216Metric_Pad1.42x1.75mm_HandSolder
- LED8: renamed from LED7; footprint MOUSER:LEDC3216X120N -> LED_SMD:LED_1206_3216Metric_Pad1.42x1.75mm_HandSolder
- LED9: renamed from LED11; footprint MOUSER:LEDC3216X120N -> LED_SMD:LED_1206_3216Metric_Pad1.42x1.75mm_HandSolder
- Q1: value BC817-25LT1G -> BC817; footprint MOUSER:SOT96P237X111-3N -> Package_TO_SOT_SMD:SOT-23
- R15: renamed from R14; value 3300 -> 300; footprint Resistor_SMD:R_0603_1608Metric -> Resistor_SMD:R_1206_3216Metric
- R7: renamed from R15; value 300 -> 270
- SW1: renamed from SW3; value SW_Push_45deg -> Switch
- SW10: renamed from SW1; value SW_Push_45deg -> Switch
- SW11: renamed from SW9; value SW_Push_45deg -> Switch
- SW12: renamed from SW10; value SW_Push_45deg -> Switch
- SW13: renamed from SW11; value SW_Push_45deg -> Switch
- SW14: renamed from SW12; value SW_Push_45deg -> Switch
- SW15: renamed from SW13; value SW_Push_45deg -> Switch
- SW16: renamed from SW21; value SW_Push_45deg -> Switch
- SW17: renamed from SW14; value SW_Push_45deg -> Switch
- SW18: renamed from SW22; value SW_Push_45deg -> Switch
- SW19: renamed from SW23; value SW_Push_45deg -> Switch
- SW2: renamed from SW4; value SW_Push_45deg -> Switch
- SW20: renamed from SW29; value SW_Push_45deg -> Switch
- SW21: renamed from SW31; value SW_Push_45deg -> Switch
- SW22: renamed from SW34; value SW_Push_45deg -> Switch
- SW23: renamed from SW2; value SW_Push_45deg -> Switch
- SW24: renamed from SW15; value SW_Push_45deg -> Switch
- SW25: renamed from SW16; value SW_Push_45deg -> Switch
- SW26: renamed from SW17; value SW_Push_45deg -> Switch
- SW27: renamed from SW18; value SW_Push_45deg -> Switch
- SW28: renamed from SW19; value SW_Push_45deg -> Switch
- SW29: renamed from SW20; value SW_Push_45deg -> Switch
- SW3: renamed from SW5; value SW_Push_45deg -> Switch
- SW30: renamed from SW24; value SW_Push_45deg -> Switch
- SW31: renamed from SW25; value SW_Push_45deg -> Switch
- SW32: renamed from SW26; value SW_Push_45deg -> Switch
- SW33, SW35: value SW_Push_45deg -> Switch
- SW4: renamed from SW6; value SW_Push_45deg -> Switch
- SW5: renamed from SW7; value SW_Push_45deg -> Switch
- SW6: renamed from SW8; value SW_Push_45deg -> Switch
- SW8: renamed from SW28; value SW_Push_45deg -> Switch
- moved LED1 226.0 mm to (252.7, 32.3)
- moved LED2 224.5 mm to (252.6, 51.6)
- moved R1 221.4 mm to (252.6, 38.2), turned to -90 degrees
- moved R2 220.2 mm to (252.6, 45.4), turned to 90 degrees
- moved R12 217.8 mm to (42.0, 35.4)
- moved R10 195.3 mm to (62.6, 38.1), turned to 90 degrees
- moved LED10 195.1 mm to (66.6, 37.9)
- moved LED11 177.9 mm to (84.0, 54.6)
- moved LED12 172.1 mm to (47.4, 35.6)
- moved LED4 154.6 mm to (215.2, 59.6)
- moved R4 153.2 mm to (210.0, 59.7)
- moved LED3 152.9 mm to (213.0, 30.2)
- moved R3 152.1 mm to (208.4, 30.4), turned to 90 degrees
- moved LED9 135.7 mm to (98.4, 54.8), turned to 90 degrees
- moved R11 133.9 mm to (80.2, 54.4), turned to 90 degrees
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- renumbered R2 to R1, R13 to R10, R10 to R11, R8 to R13, R1 to R2, R4 to R3, R3 to R4, R9 to R5, R5 to R6, R11 to R8, R7 to R9
Connections:
- D1 pad 2: Net-(D5-A) -> Net-(D1-A)
- D10 pad 1: ROW2 -> ROW1
- D10 pad 2: Net-(D15-A) -> Net-(D10-A)
- D11 pad 1: ROW2 -> ROW1
- D11 pad 2: Net-(D16-A) -> Net-(D11-A)
- D12 pad 2: Net-(D11-A) -> Net-(D12-A)
- D13 pad 1: ROW2 -> ROW1
- D13 pad 2: Net-(D18-A) -> Net-(D13-A)
- D14 pad 1: ROW2 -> ROW1
- D14 pad 2: Net-(D17-A) -> Net-(D14-A)
- D15 pad 2: Net-(D12-A) -> Net-(D15-A)
- D16 pad 1: ROW2 -> ROW1
- D16 pad 2: Net-(D19-A) -> Net-(D16-A)
- D17 pad 2: Net-(D13-A) -> Net-(D17-A)
- D18 pad 2: Net-(D14-A) -> Net-(D18-A)
- D19 pad 1: ROW0 -> ROW1
- D19 pad 2: Net-(D8-A) -> Net-(D19-A)
- D2 pad 1: ROW1 -> ROW0
- D20 pad 1: ROW0 -> ROW1
- D20 pad 2: Net-(D28-A) -> Net-(D20-A)
- D21 pad 1: ROW0 -> ROW1
- D21 pad 2: Net-(D30-A) -> Net-(D21-A)
- D22 pad 1: ROW0 -> ROW1
- D22 pad 2: Net-(D27-A) -> Net-(D22-A)
- D23 pad 2: Net-(D20-A) -> Net-(D23-A)
- D25 pad 1: ROW1 -> ROW2
- D25 pad 2: Net-(D21-A) -> Net-(D25-A)
- D26 pad 2: Net-(D25-A) -> Net-(D26-A)
- D27 pad 1: ROW1 -> ROW2
- D27 pad 2: Net-(D23-A) -> Net-(D27-A)
- D28 pad 1: ROW1 -> ROW2
- D28 pad 2: Net-(D22-A) -> Net-(D28-A)
- D29 pad 1: ROW1 -> ROW2
- D3 pad 1: ROW1 -> ROW0
- D3 pad 2: Net-(D10-A) -> Net-(D3-A)
- D30 pad 2: Net-(D32-A) (its old number) -> Net-(D30-A)
- D31 pad 1: ROW1 -> ROW2
- D33 pad 2: Net-(D35-A) -> Net-(D33-A)
- D34 pad 1: ROW1 -> ROW2
- D35 pad 2: Net-(D33-A) -> Net-(D35-A)
- D4 pad 2: Net-(D3-A) -> Net-(D4-A)
- D5 pad 2: Net-(D4-A) -> Net-(D5-A)
- D6 pad 2: Net-(D1-A) -> Net-(D6-A)
- D7 pad 1: ROW1 -> ROW0
- D7 pad 2: Net-(D9-A) -> Net-(D7-A)
- D8 pad 2: Net-(D6-A) -> Net-(D8-A)
- D9 pad 2: Net-(D7-A) -> Net-(D9-A)
- LED11 pad 2: Net-(LED12-A) -> Net-(LED11-A)
- LED12 pad 2: Net-(LED10-A) (its old number) -> Net-(LED12-A)
- LED13 pad 2: Net-(LED6-A) (its old number) -> Net-(LED13-A)
- LED7 pad 1: GND -> Net-(LED1-K)
- LED8 pad 2: Net-(LED7-A) (its old number) -> Net-(LED8-A)
- LED9 pad 2: Net-(LED11-A) -> Net-(LED9-A)
- R11 pad 1: Net-(LED10-A) (its old number) -> Net-(LED11-A)
- R13 pad 1: Net-(LED8-A) -> Net-(LED13-A)
- R15 pad 1: LED -> Net-(LED15-A)
- R15 pad 2: Net-(Q1-B) -> LED_MC
- R7 pad 2: LED_MC -> 5V
- R8 pad 1: Net-(LED11-A) -> Net-(LED8-A)
- R9 pad 1: Net-(LED7-A) (its old number) -> Net-(LED9-A)
- SW1 pad 2: Net-(D3-A) -> Net-(D1-A)
- SW10 pad 2: Net-(D1-A) -> Net-(D10-A)
- SW11 pad 2: Net-(D9-A) -> Net-(D11-A)
- SW12 pad 2: Net-(D10-A) -> Net-(D12-A)
- SW13 pad 2: Net-(D11-A) -> Net-(D13-A)
- SW14 pad 2: Net-(D12-A) -> Net-(D14-A)
- SW15 pad 2: Net-(D13-A) -> Net-(D15-A)
- SW16 pad 1: COL7 -> COL6
- SW16 pad 2: Net-(D21-A) -> Net-(D16-A)
- SW17 pad 1: COL6 -> COL7
- SW17 pad 2: Net-(D14-A) -> Net-(D17-A)
- SW18 pad 2: Net-(D22-A) -> Net-(D18-A)
- SW19 pad 2: Net-(D23-A) -> Net-(D19-A)
- SW2 pad 2: Net-(D4-A) -> Net-(D2-A)
- SW20 pad 2: Net-(D29-A) -> Net-(D20-A)
- SW21 pad 2: Net-(D31-A) -> Net-(D21-A)
- SW22 pad 2: Net-(D34-A) -> Net-(D22-A)
- SW23 pad 2: Net-(D2-A) -> Net-(D23-A)
- SW24 pad 1: COL0 -> COL1
- SW24 pad 2: Net-(D15-A) -> Net-(D24-A)
- SW25 pad 1: COL1 -> COL2
- SW25 pad 2: Net-(D16-A) -> Net-(D25-A)
- SW26 pad 1: COL2 -> COL3
- SW26 pad 2: Net-(D17-A) -> Net-(D26-A)
- SW27 pad 1: COL3 -> COL4
- SW27 pad 2: Net-(D18-A) -> Net-(D27-A)
- SW28 pad 1: COL4 -> COL5
- SW28 pad 2: Net-(D19-A) -> Net-(D28-A)
- SW29 pad 1: COL5 -> COL6
- SW29 pad 2: Net-(D20-A) -> Net-(D29-A)
- SW3 pad 2: Net-(D5-A) -> Net-(D3-A)
- SW30 pad 1: COL6 -> COL7
- SW30 pad 2: Net-(D24-A) -> Net-(D30-A)
- SW31 pad 1: COL7 -> COL8
- SW31 pad 2: Net-(D25-A) -> Net-(D31-A)
- SW32 pad 1: COL8 -> COL9
- SW35 pad 1: COL11 -> COL12
- SW4 pad 2: Net-(D6-A) -> Net-(D4-A)
- SW5 pad 2: Net-(D7-A) -> Net-(D5-A)
- SW6 pad 2: Net-(D8-A) -> Net-(D6-A)
- SW8 pad 1: COL8 -> COL10
- SW8 pad 2: Net-(D28-A) -> Net-(D8-A)
Routing:
- net LED: track 34.1 -> 197.1 mm
- net COL0: track 174.9 -> 62.1 mm
- net GND: track 62.4 -> 170.9 mm
- net COL1: track 159.1 -> 61.1 mm
- net COL10: track 91.8 -> 179.6 mm, vias 1 -> 0
- net COL11: track 101.4 -> 187.5 mm, vias 3 -> 0
- net COL12: track 104.9 -> 186.8 mm, vias 1 -> 0
- net COL2: track 138.4 -> 56.8 mm
- net Net-(LED1-K): track 438.4 -> 362.2 mm, vias 2 -> 5
- net COL3: track 124.8 -> 56.7 mm, vias 1 -> 0
- net LED_MC: track 32.4 -> 91.8 mm
- net 5V: track 414.2 -> 357.5 mm, vias 6 -> 9
- net COL8: track 86.2 -> 137.0 mm
- net ROW0: track 241.1 -> 283.5 mm, vias 2 -> 0
- net COL6: track 71.8 -> 104.1 mm
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Other:
- outline, holes or cut-outs redrawn
- board text removed: "ROW0 ROW2 COL1 COL3 COL5 COL7 COL9 COL11 LED GND"
- board text removed: "ROW1 COL0 COL2 COL4 COL6 COL8 COL10 COL12 LEDMC 5V"

Commit message: feat: now using 4 layer pcb
Parts:
- moved R15 17.3 mm to (192.2, 33.6), turned to -90 degrees
- moved LED15 15.9 mm to (192.2, 28.6), turned to -90 degrees
- moved Q1 10.6 mm to (260.5, 30.0), turned to 180 degrees
- moved R16 3.97 mm to (264.8, 31.2), turned to 180 degrees
- moved R13 2.48 mm to (42.4, 53.6), turned to 90 degrees
- moved LED13 2.20 mm to (47.4, 53.6), turned to -90 degrees
- turned LED4 to -90 degrees
Routing:
- net Net-(LED1-K): track 362.2 -> 313.4 mm, vias 5 -> 0
- net ROW0: track 283.5 -> 241.1 mm, vias 0 -> 1
- net ROW1: track 306.7 -> 267.3 mm, vias 0 -> 1
- net 5V: track 357.5 -> 332.6 mm, vias 9 -> 3
- net ROW2: track 269.8 -> 245.4 mm
- net LED_MC: track 91.8 -> 106.8 mm
- net LED: track 197.1 -> 187.5 mm, vias 0 -> 1
- net Net-(Q1-B): track 11.5 -> 2.66 mm, vias 1 -> 0
- net GND: track 170.9 -> 178.5 mm, vias 1 -> 2
- net Net-(LED15-A): track 7.94 -> 2.05 mm
- net COL2: track 56.8 -> 51.9 mm
- net COL6: track 104.1 -> 102.1 mm
- net Net-(D30-A): track 11.7 -> 10.1 mm
- net COL0: track 62.1 -> 60.9 mm
- net Net-(LED4-A): track 5.25 -> 6.40 mm
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Other:
- copper layers 2 -> 4
- board text added: "A10C UFC PCB v1.1.0 made by w3z315 (michler.io)"
- board text added: "GND +5V"
- board text added: "LED_MC"
- board text added: "ROW0 ROW1 ROW2 COL0 COL1 COL2 COL3 COL4 COL5 COL6 COL7 COL8 COL9 COL10 COL11 COL12 LED"
- board text removed: "A10C UFC PCB v1.0.0 made by w3z315 (michler.io)"
